File: MegaCD-Connect BD Remake.kicad_pcb (KiCad board)
At the start: 2 copper layers, 98 x 44 mm, 17 parts, among them IC1 GAL22V10, IC2 74HC374, IC3 74HC374, IC4 74ACT10, IC5 74HC245, IC6 74HC245, J1 MD EXPANSION, J2 CD EXPANSION, J3 TREE HOUSE

Commit message: Add files via upload
Parts:
- added C7: 22uF, Capacitor_Tantalum_SMD:CP_EIA-3528-12_Kemet-T_Pad1.50x2.35mm_HandSolder, F.Cu at (119.9, 85.1)
- moved J3 2.29 mm to (118.4, 92.1)
- moved C2 1.22 mm to (146.2, 102.4), turned to 180 degrees
- moved C4 1.06 mm to (128.5, 90.8)
- moved C1 0.46 mm to (114.3, 102.4)
- moved C5 0.38 mm to (147.8, 90.8)
- moved C3 0.33 mm to (174.8, 102.4)
- moved C6 0.18 mm to (175.3, 90.8)
Connections:
- J2 pad a26: VCC -> +9V
- J2 pad a28: +9V -> unconnected-(J2-Pin_a28-Pada28)
- J2 pad b26: VCC -> +9V
- J2 pad b28: +9V -> unconnected-(J2-Pin_b28-Padb28)
Routing:
- net /VA17: track 101.9 -> 35.9 mm
- net /VA7: track 96.7 -> 37.7 mm, vias 1 -> 0
- net TR_CE: track 68.0 -> 119.6 mm, vias 0 -> 1
- net TR_CP: track 79.7 -> 127.8 mm, vias 0 -> 4
- net TR_DIR: track 51.5 -> 95.6 mm, vias 2 -> 1
- net /VA2: track 39.2 -> 82.7 mm
- net /VA6: track 82.6 -> 40.5 mm
- net /VA4: track 35.7 -> 74.5 mm, vias 0 -> 4
- net /VD14: track 31.0 -> 67.8 mm, vias 1 -> 2
- net /VD6: track 35.6 -> 60.2 mm
- net ~{CAS2}: track 76.9 -> 52.5 mm
- net ~{ASEL}: track 50.5 -> 73.7 mm, vias 1 -> 2
- net FRES: track 57.4 -> 35.9 mm
- net /VD12: track 33.6 -> 54.1 mm, vias 1 -> 2
- net ~{CAS0}: track 83.9 -> 102.3 mm, vias 1 -> 2
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Other:
- board text added: "JRBVZ 2025"
