File: MegaCD-Connect BD Remake.kicad_sch (KiCad schematic)
At the start: 17 parts, among them IC1 GAL22V10, IC2 74HC374, IC3 74HC374, IC4 74ACT10, IC5 74HC245, IC6 74HC245, J1 MD EXPANSION, J2 CD EXPANSION, J3 TREE HOUSE

Commit message: Add files via upload
Parts:
- added C7: 22uF, Capacitor_Tantalum_SMD:CP_EIA-3528-12_Kemet-T_Pad1.50x2.35mm_HandSolder, symbol Device:C_Polarized
Connections:
- net +9V: now also J2.a26 (Pin_a26), J2.b26 (Pin_b26); no longer J2.a28 (Pin_a28), J2.b28 (Pin_b28)
- net GND: now also C7.2
- net VCC: now also C7.1; no longer J2.a26 (Pin_a26), J2.b26 (Pin_b26)
- no-connect marks 12 -> 14
